File: main.sch (KiCad schematic (older format))
At the start: 23 parts, among them J1 USB_OTG, J2 MCS-48 PINS, J3 SPI, J4 EXT2, J5 EXT1, SW1 SW_SPST, U1 LTC4415, U2 STF202-22, U5 AT90USB1286-AU, Y1 16Mhz

Commit message: cleaned up pcb, added status LEDs
Parts:
- added D1, D2: PWR, LEDs:LED_0402, symbol LED_Small_ALT
- added R4, R5: 250, Resistors_SMD:R_0402, symbol R_Small
Connections:
- net +5VD: now also D1.2 (A)
- net GNDD: now also R4.1, R5.1
- net ON: now reaches J5.4 (Pin_4), U5.34 (PE1)
- net ON: now also D2.2 (A)
- new net: D1.1 (K), R4.2
- new net: D2.1 (K), R5.2
Changed lines of the file:
@@
 Wire Wire Line
 	8690 3290 9130 3290
-Wire Wire Line
-	9130 2990 9070 2990
-Wire Wire Line
-	9070 2990 9070 5190
-Wire Wire Line
-	9070 5190 6620 5190
-Wire Wire Line
-	6620 5190 6620 3190
-Wire Wire Line
-	6620 3190 7490 3190
 $Comp
 L Conn_01x03 J4
@@
 	1    0    0    -1
 $EndComp
+$Comp
+L LED_Small_ALT D1
+U 1 1 5CA1D670
+P 2410 3840
+F 0 "D1" H 2430 3740 50  0000 L CNN
+F 1 "PWR" H 2235 3740 50  0000 L CNN
+F 2 "LEDs:LED_0402" V 2410 3840 50  0001 C CNN
+F 3 "" V 2410 3840 50  0001 C CNN
+	1    2410 3840
+	1    0    0    -1
+$EndComp
+$Comp
+L R_Small R4
+U 1 1 5CA1D897
+P 2210 3840
+F 0 "R4" V 2290 3770 50  0000 L CNN
+F 1 "250" V 2210 3760 50  0000 L CNN
+F 2 "Resistors_SMD:R_0402" H 2210 3840 50  0001 C CNN
+F 3 "" H 2210 3840 50  0001 C CNN
+	1    2210 3840
+	0    -1   -1   0
+$EndComp
+$Comp
+L GNDD #PWR029
+U 1 1 5CA1D9A0
+P 2110 3840
+F 0 "#PWR029" H 2110 3590 50  0001 C CNN
+F 1 "GNDD" H 2110 3715 50  0000 C CNN
+F 2 "" H 2110 3840 50  0001 C CNN
+F 3 "" H 2110 3840 50  0001 C CNN
+	1    2110 3840
+	1    0    0    -1
+$EndComp
+$Comp
+L +5VD #PWR030
+U 1 1 5CA1DB27
+P 2510 3840
+F 0 "#PWR030" H 2510 3690 50  0001 C CNN
+F 1 "+5VD" H 2510 3980 50  0000 C CNN
+F 2 "" H 2510 3840 50  0001 C CNN
+F 3 "" H 2510 3840 50  0001 C CNN
+	1    2510 3840
+	1    0    0    -1
+$EndComp
+$Comp
+L LED_Small_ALT D2
+U 1 1 5CA1DE3B
+P 2410 4170
+F 0 "D2" H 2430 4070 50  0000 L CNN
+F 1 "PWR" H 2235 4070 50  0000 L CNN
+F 2 "LEDs:LED_0402" V 2410 4170 50  0001 C CNN
+F 3 "" V 2410 4170 50  0001 C CNN
+	1    2410 4170
+	1    0    0    -1
+$EndComp
+$Comp
+L R_Small R5
+U 1 1 5CA1DE41
+P 2210 4170
+F 0 "R5" V 2290 4100 50  0000 L CNN
+F 1 "250" V 2210 4090 50  0000 L CNN
+F 2 "Resistors_SMD:R_0402" H 2210 4170 50  0001 C CNN
+F 3 "" H 2210 4170 50  0001 C CNN
+	1    2210 4170
+	0    -1   -1   0
+$EndComp
+$Comp
+L GNDD #PWR031
+U 1 1 5CA1DE47
+P 2110 4170
+F 0 "#PWR031" H 2110 3920 50  0001 C CNN
+F 1 "GNDD" H 2110 4045 50  0000 C CNN
+F 2 "" H 2110 4170 50  0001 C CNN
+F 3 "" H 2110 4170 50  0001 C CNN
+	1    2110 4170
+	1    0    0    -1
+$EndComp
+Text Label 7490 3190 2    60   ~ 0
+ON
+Text Label 2510 4170 0    60   ~ 0
+ON
+Text Label 9130 2990 2    60   ~ 0
+ON
 $EndSCHEMATC

Commit message: legal shenanigans
Other:
- note added: "Copyright Listofoptions (James M.) 2019.\nThis documentation describes Open Hardware and is licensed under the\nCERN OHL v. 1.2. You may redistribute and modify this documentation under the\nterms of the CERN OHL v.1.2. (http://ohwr.org/cernohl). This documentation is\ndistributed WITHOUT ANY EXPRESS OR IMPLIED WARRANTY,INCLUDING OF\nMERCHANTABILITY, SATISFACTORY QUALITY AND FITNESS FOR A PARTICU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"
Changed lines of the file:
@@
 LIBS:MCU_Microchip_AVR
 LIBS:analog_devices
-LIBS:_div
+LIBS:ltc4415
 LIBS:main-cache
 EELAYER 25 0
@@
 $EndComp
 $Comp
-L LTC4415 U1
-U 1 1 5CA2B328
-P 2440 2770
-F 0 "U1" H 2790 3270 60  0000 C CNN
-F 1 "LTC4415" H 2190 3270 60  0000 C CNN
-F 2 "Housings_DFN_QFN:DFN-16-1EP_3x5mm_Pitch0.5mm" H 2440 2820 60  0001 C CNN
-F 3 "" H 2440 2820 60  0000 C CNN
-	1    2440 2770
-	1    0    0    -1
-$EndComp
-$Comp
 L GNDD #PWR014
 U 1 1 5CA2B8DF
@@
 Text Label 9130 2990 2    60   ~ 0
 ON
+Text Notes 470  7800 0    60   ~ 0
+Copyright Listofoptions (James M.) 2019.\nThis documentation describes Open Hardware and is licensed under the\nCERN OHL v. 1.2. You may redistribute and modify this documentation under the\nterms of the CERN OHL v.1.2. (http://ohwr.org/cernohl). This documentation is\ndistributed WITHOUT ANY EXPRESS OR IMPLIED WARRANTY,INCLUDING OF\nMERCHANTABILITY, SATISFACTORY QUALITY AND FITNESS FOR A PARTICULAR PURPOSE.\nPlease see the CERN OHL v.1.2 for applicable conditions
+$Comp
+L LTC4415 U1
+U 1 1 5CA24DB7
+P 2440 2770
+F 0 "U1" H 2790 3270 60  0000 C CNN
+F 1 "LTC4415" H 2190 3270 60  0000 C CNN
+F 2 "Housings_DFN_QFN:DFN-16-1EP_3x5mm_Pitch0.5mm" H 2440 2820 60  0001 C CNN
+F 3 "" H 2440 2820 60  0000 C CNN
+	1    2440 2770
+	1    0    0    -1
+$EndComp
 $EndSCHEMATC

Commit message: improved groundplane, and used beefier supply caps
Parts:
- C10, C8, C9: value 4u7 -> 100u; footprint Capacitors_SMD:C_0201 -> Capacitors_SMD:C_0805
Connections:
- no-connect marks 2 -> 3
Changed lines of the file:
@@
 P 2080 1840
 F 0 "C8" H 2090 1770 50  0000 L CNN
-F 1 "4u7" H 1920 1780 50  0000 L CNN
-F 2 "Capacitors_SMD:C_0201" H 2080 1840 50  0001 C CNN
+F 1 "100u" H 1870 1780 50  0000 L CNN
+F 2 "Capacitors_SMD:C_0805" H 2080 1840 50  0001 C CNN
 F 3 "" H 2080 1840 50  0001 C CNN
 	1    2080 1840
@@
 $EndComp
 $Comp
-L C_Small C9
-U 1 1 5CA2D65D
-P 2390 1840
-F 0 "C9" H 2400 1770 50  0000 L CNN
-F 1 "4u7" H 2230 1780 50  0000 L CNN
-F 2 "Capacitors_SMD:C_0201" H 2390 1840 50  0001 C CNN
-F 3 "" H 2390 1840 50  0001 C CNN
-	1    2390 1840
-	1    0    0    -1
-$EndComp
-$Comp
 L GNDD #PWR023
 U 1 1 5CA2D669
@@
 P 2690 1840
 F 0 "C10" H 2700 1770 50  0000 L CNN
-F 1 "4u7" H 2530 1780 50  0000 L CNN
-F 2 "Capacitors_SMD:C_0201" H 2690 1840 50  0001 C CNN
+F 1 "100u" H 2500 1780 50  0000 L CNN
+F 2 "Capacitors_SMD:C_0805" H 2690 1840 50  0001 C CNN
 F 3 "" H 2690 1840 50  0001 C CNN
 	1    2690 1840
@@
 	1    0    0    -1
 $EndComp
+$Comp
+L C_Small C9
+U 1 1 5CA2D65D
+P 2390 1840
+F 0 "C9" H 2400 1770 50  0000 L CNN
+F 1 "100u" H 2200 1780 50  0000 L CNN
+F 2 "Capacitors_SMD:C_0805" H 2390 1840 50  0001 C CNN
+F 3 "" H 2390 1840 50  0001 C CNN
+	1    2390 1840
+	1    0    0    -1
+$EndComp
+NoConn ~ 4480 1940
 $EndSCHEMATC

Commit message: shenanigans and bootloader jumper on clock xtal-1 pin
Parts:
- added JP1: BOOT, Resistors_SMD:R_0201_NoSilk, symbol Jumper_NO_Small
Connections:
- net XTAL+: now also JP1.2; no longer C2.2, Y1.4
- new net: C2.2, JP1.1, Y1.4
Changed lines of the file:
@@
 	1    0    0    -1
 $EndComp
-Wire Wire Line
-	4180 2140 4180 2190
-Wire Wire Line
-	4080 2140 4180 2140
-Wire Wire Line
-	1550 2670 1550 2420
-Connection ~ 1790 2970
-Wire Wire Line
-	1310 2970 1310 2420
-Wire Wire Line
-	1790 2970 1310 2970
-Wire Wire Line
-	1790 2920 1790 3020
-Wire Wire Line
-	1240 3170 1240 3270
-Wire Wire Line
-	1790 3170 1240 3170
-Wire Wire Line
-	1510 3270 1790 3270
-Wire Wire Line
-	1790 3470 1790 3420
-Connection ~ 1790 2670
-Wire Wire Line
-	1550 2670 1790 2670
-Connection ~ 3090 2420
-Connection ~ 1790 2420
-Connection ~ 3090 2670
-Connection ~ 3090 2520
-Wire Wire Line
-	3090 2420 3090 2770
-Wire Wire Line
-	1790 2670 1790 2770
-Wire Wire Line
-	1790 2520 1790 2420
-Wire Wire Line
-	5380 1840 5380 2290
-Wire Wire Line
-	4480 1840 5380 1840
-Wire Wire Line
-	4480 1740 5290 1740
-Wire Wire Line
-	7210 2290 7020 2290
-Wire Wire Line
-	7210 2340 7210 2290
-Wire Wire Line
-	7300 2340 7210 2340
-Wire Wire Line
-	7300 2390 7300 2340
-Wire Wire Line
-	7490 2390 7300 2390
-Wire Wire Line
-	7260 2290 7490 2290
-Wire Wire Line
-	7260 2390 7260 2290
-Wire Wire Line
-	7020 2390 7260 2390
-Wire Wire Line
-	6330 1110 6330 1860
-Wire Wire Line
-	6330 1110 6500 1110
-Wire Wire Line
-	6500 1110 6500 1140
-Wire Wire Line
-	6330 1860 6500 1860
-Wire Wire Line
-	6500 1860 6500 1840
-Wire Wire Line
-	6500 1590 6500 1640
-Wire Wire Line
-	6500 1340 6500 1390
-Wire Wire Line
-	6500 1370 7490 1370
-Connection ~ 6500 1370
-Wire Wire Line
-	7490 1630 6500 1630
-Connection ~ 6500 1630
-Wire Wire Line
-	6300 1490 6300 1910
-Wire Wire Line
-	6300 1910 7490 1910
-Wire Wire Line
-	6670 1490 6670 1910
-Connection ~ 6300 1490
-Wire Wire Line
-	8070 5670 7900 5670
-Wire Wire Line
-	7900 5950 8070 5950
-Wire Wire Line
-	7900 6230 8070 6230
-Connection ~ 7900 5950
-Wire Wire Line
-	8070 5470 8310 5470
-Wire Wire Line
-	8310 6030 8070 6030
-Wire Wire Line
-	8070 5750 8310 5750
-Connection ~ 8310 5750
-Connection ~ 8310 5470
-Wire Wire Line
-	7250 2850 7050 2850
-Wire Wire Line
-	7050 2850 7050 2190
-Wire Wire Line
-	7050 2190 7020 2190
-Wire Wire Line
-	5870 1860 5870 2190
-Wire Wire Line
-	5870 1990 7490 1990
-Wire Wire Line
-	7490 1990 7490 2090
-Connection ~ 5870 1990
-Wire Wire Line
-	5640 1910 5870 1910
-Connection ~ 5870 1910
-Wire Wire Line
-	5380 2290 5870 2290
-Wire Wire Line
-	5290 2390 5870 2390
-Wire Wire Line
-	7250 2590 7490 2590
-Wire Wire Line
-	7490 1630 7490 1690
-Wire Wire Line
-	7490 1370 7490 1490
-Wire Wire Line
-	6700 1290 7490 1290
-Wire Wire Line
-	8310 5470 8310 6030
-Wire Wire Line
-	7900 5670 7900 6230
-Connection ~ 7900 6230
-Wire Wire Line
-	7990 4990 8090 4990
-Connection ~ 8090 4990
-Wire Wire Line
-	7990 990  8190 990
-Connection ~ 8090 990
-Wire Wire Line
-	7490 1910 7490 1890
-Connection ~ 6670 1910
-Wire Wire Line
-	5290 1740 5290 2390
-Wire Wire Line
-	7250 2850 7250 2790
-Connection ~ 7050 2850
-Wire Wire Line
-	8690 2190 9120 2190
-Wire Wire Line
-	8690 2290 9120 2290
-Wire Wire Line
-	8690 2390 9120 2390
-Wire Wire Line
-	8690 2490 9120 2490
-Wire Wire Line
-	7490 3290 7230 3290
-Wire Wire Line
-	6900 3290 7030 3290
-Wire Wire Line
-	6170 1490 6670 1490
-Wire Wire Line
-	6700 850  6700 1290
-Wire Wire Line
-	6790 850  6700 850
-Wire Wire Line
-	7190 850  7280 850
-Connection ~ 4180 2140
-Connection ~ 6330 1490
-Connection ~ 6380 1490
-Connection ~ 6620 1490
-Wire Wire Line
-	3090 3070 3090 3470
-Connection ~ 3090 3170
-Connection ~ 3090 3320
 $Comp
 L GNDD #PWR028
@@
 	1    0    0    -1
 $EndComp
-Connection ~ 3090 3420
 $Comp
 L Conn_01x04 J5
@@
 	1    0    0    1
 $EndComp
-Wire Wire Line
-	8690 3090 9130 3090
-Wire Wire Line
-	8690 3190 9130 3190
-Wire Wire Line
-	8690 3290 9130 3290
 $Comp
 L Conn_01x03 J4
@@
 	-1   0    0    1
 $EndComp
-Wire Wire Line
-	7160 3990 7490 3990
-Wire Wire Line
-	7160 4090 7490 4090
-Wire Wire Line
-	7160 4190 7490 4190
 $Comp
 L C_Small C10
@@
 $EndComp
 NoConn ~ 4480 1940
+Wire Wire Line
+	4180 2140 4180 2190
+Wire Wire Line
+	4080 2140 4180 2140
+Wire Wire Line
+	1550 2670 1550 2420
+Connection ~ 1790 2970
+Wire Wire Line
+	1310 2970 1310 2420
+Wire Wire Line
+	1790 2970 1310 2970
+Wire Wire Line
+	1790 2920 1790 3020
+Wire Wire Line
+	1240 3170 1240 3270
+Wire Wire Line
+	1790 3170 1240 3170
+Wire Wire Line
+	1510 3270 1790 3270
+Wire Wire Line
+	1790 3470 1790 3420
+Connection ~ 1790 2670
+Wire Wire Line
+	1550 2670 1790 2670
+Connection ~ 3090 2420
+Connection ~ 1790 2420
+Connection ~ 3090 2670
+Connection ~ 3090 2520
+Wire Wire Line
+	3090 2420 3090 2770
+Wire Wire Line
+	1790 2670 1790 2770
+Wire Wire Line
+	1790 2520 1790 2420
+Wire Wire Line
+	5380 1840 5380 2290
+Wire Wire Line
+	4480 1840 5380 1840
+Wire Wire Line
+	4480 1740 5290 1740
+Wire Wire Line
+	7210 2290 7020 2290
+Wire Wire Line
+	7210 2340 7210 2290
+Wire Wire Line
+	7300 2340 7210 2340
+Wire Wire Line
+	7300 2390 7300 2340
+Wire Wire Line
+	7490 2390 7300 2390
+Wire Wire Line
+	7260 2290 7490 2290
+Wire Wire Line
+	7260 2390 7260 2290
+Wire Wire Line
+	7020 2390 7260 2390
+Wire Wire Line
+	6330 1110 6330 1860
+Wire Wire Line
+	6330 1110 6500 1110
+Wire Wire Line
+	6500 1110 6500 1140
+Wire Wire Line
+	6330 1860 6500 1860
+Wire Wire Line
+	6500 1860 6500 1840
+Wire Wire Line
+	6500 1590 6500 1640
+Wire Wire Line
+	6500 1340 6500 1390
+Connection ~ 6500 1370
+Wire Wire Line
+	7490 1630 6500 1630
+Connection ~ 6500 1630
+Wire Wire Line
+	6300 1490 6300 1910
+Wire Wire Line
+	6300 1910 7490 1910
+Wire Wire Line
+	6670 1490 6670 1910
+Connection ~ 6300 1490
+Wire Wire Line
+	8070 5670 7900 5670
+Wire Wire Line
+	7900 5950 8070 5950
+Wire Wire Line
+	7900 6230 8070 6230
+Connection ~ 7900 5950
+Wire Wire Line
+	8070 5470 8310 5470
+Wire Wire Line
+	8310 6030 8070 6030
+Wire Wire Line
+	8070 5750 8310 5750
+Connection ~ 8310 5750
+Connection ~ 8310 5470
+Wire Wire Line
+	7250 2850 7050 2850
+Wire Wire Line
+	7050 2850 7050 2190
+Wire Wire Line
+	7050 2190 7020 2190
+Wire Wire Line
+	5870 1860 5870 2190
+Wire Wire Line
+	5870 1990 7490 1990
+Wire Wire Line
+	7490 1990 7490 2090
+Connection ~ 5870 1990
+Wire Wire Line
+	5640 1910 5870 1910
+Connection ~ 5870 1910
+Wire Wire Line
+	5380 2290 5870 2290
+Wire Wire Line
+	5290 2390 5870 2390
+Wire Wire Line
+	7250 2590 7490 2590
+Wire Wire Line
+	7490 1630 7490 1690
+Wire Wire Line
+	7490 1370 7490 1490
+Wire Wire Line
+	6700 1290 7490 1290
+Wire Wire Line
+	8310 5470 8310 6030
+Wire Wire Line
+	7900 5670 7900 6230
+Connection ~ 7900 6230
+Wire Wire Line
+	7990 4990 8090 4990
+Connection ~ 8090 4990
+Wire Wire Line
+	7990 990  8190 990
+Connection ~ 8090 990
+Wire Wire Line
+	7490 1910 7490 1890
+Connection ~ 6670 1910
+Wire Wire Line
+	5290 1740 5290 2390
+Wire Wire Line
+	7250 2850 7250 2790
+Connection ~ 7050 2850
+Wire Wire Line
+	8690 2190 9120 2190
+Wire Wire Line
+	8690 2290 9120 2290
+Wire Wire Line
+	8690 2390 9120 2390
+Wire Wire Line
+	8690 2490 9120 2490
+Wire Wire Line
+	7490 3290 7230 3290
+Wire Wire Line
+	6900 3290 7030 3290
+Wire Wire Line
+	6170 1490 6670 1490
+Wire Wire Line
+	6700 850  6700 1290
+Wire Wire Line
+	6790 850  6700 850
+Wire Wire Line
+	7190 850  7280 850
+Connection ~ 4180 2140
+Connection ~ 6330 1490
+Connection ~ 6380 1490
+Connection ~ 6620 1490
+Wire Wire Line
+	3090 3070 3090 3470
+Connection ~ 3090 3170
+Connection ~ 3090 3320
+Connection ~ 3090 3420
+Wire Wire Line
+	8690 3090 9130 3090
+Wire Wire Line
+	8690 3190 9130 3190
+Wire Wire Line
+	8690 3290 9130 3290
+Wire Wire Line
+	7160 3990 7490 3990
+Wire Wire Line
+	7160 4090 7490 4090
+Wire Wire Line
+	7160 4190 7490 4190
+Wire Wire Line
+	7490 1370 7120 1370
+Wire Wire Line
+	6920 1370 6500 1370
+$Comp
+L Jumper_NO_Small JP1
+U 1 1 5CA47697
+P 7020 1370
+F 0 "JP1" H 7210 1310 50  0000 C CNN
+F 1 "BOOT" H 7030 1310 50  0000 C CNN
+F 2 "Resistors_SMD:R_0201_NoSilk" H 7020 1370 50  0001 C CNN
+F 3 "" H 7020 1370 50  0001 C CNN
+	1    7020 1370
+	1    0    0    -1
+$EndComp
 $EndSCHEMATC
